File: v1/eagle/frontend_v1.sch (EAGLE design)
At the start: 57 parts, among them IC1 TINY24/44/84-SSU, IC2 AD5339MSOP8, IC3 LM4041A12DCK, Q10 TIP42C, Q9 TIP41C, T3 TIP35CVERTICAL, T4 TIP35CVERTICAL, U2 LM35DT, U3 LM35DT

Commit message: minor changes
Parts:
- R1, R16, R17, R35: device rcl:R-US_R2010 -> rcl:R-US_R2512
Other:
- moved on the sheet: C24, C25, HDR_OUT

Commit message: slight changes for board house
Parts:
- removed HEADER_ICSP: AVR_SPI_PRG_6PTH, SparkFun-Connectors:AVR_SPI_PRG_6PTH
- removed R5: 5k, rcl:R-US_M0805
- removed R6: 1k, rcl:R-US_M0805
- removed SERIAL: (no value), con-amp-quick:M02
- added C10, C8: 1u, rcl:C-USC0805
- added C11, C9: 0.1u, rcl:C-USC0805
- C1, C2, C3: value (none) -> 0.1u
- IC1: value TINY24/44/84-SSU -> ADC128D818; device avr-7:TINY24/44/84-SSU -> parts:ADC128D818
- R23: value 6.2k 0.1% -> 4k 0.1%
- R24: value 1.3k 0.1% -> 1k 0.1%
Connections:
- removed net ADC1: IC1.(PCINT1/AIN0/ADC1)PA1, R5.2, R6.1
- removed net ADC3: IC1.(PCINT3/T0/ADC3)PA3
- removed net N$10: IC1.(PCINT9/XTAL2)PB1, SERIAL.2
- removed net N$11: IC1.(PCINT10/INT0/OC0A/CKOUT)PB2, SERIAL.1
- removed net N$29: O1A.-IN, R23.2, R24.1
- removed net RESET: HEADER_ICSP.5, IC1.(PCINT11/RESET/DW)PB3
- new net VFEEDBACK: IC1.IN0, O1A.-IN, R23.2, R24.1
- net +5V: now also C8.1, IC1.V+; no longer HEADER_ICSP.2, IC1.VCC
- net CHANNEL_SELECT: now also IC1.A0; no longer IC1.(PCINT8/XTAL1/CLKI)PB0
- net GNDA: now also C10.2, C11.2, C8.2, C9.2, IC1.A1; no longer HEADER_ICSP.6, R6.2
- net I_CONTROL: now also IC1.IN5
- net I_SENSE: now also IC1.IN1; no longer IC1.(PCINT2/AIN1/ADC2)PA2
- net SCL: now also IC1.SCL; no longer HEADER_ICSP.3, IC1.(PCINT4/T1/SCL/USCK/ADC4)PA4
- net SDA: now also IC1.SDA; no longer HEADER_ICSP.4, IC1.(PCINT6/OC1A/SDA/MOSI/ADC6)PA6
- net TEMP_1: now also IC1.IN2; no longer HEADER_ICSP.1, IC1.(PCINT5/OC1B/MISO/DO/ADC5)PA5
- net TEMP_2: now also IC1.IN3; no longer IC1.(PCINT7/ICP/OC0B/ADC7)PA7
- net VDD: now also C10.1, C9.1, IC1.VREF; no longer IC1.(PCINT0/AREF/ADC0)PA0
- net VOUT: no longer R5.1
- net VREF: now also C11.1
- net V_CONTROL: now also IC1.IN4
Other:
- note added: "Vo = Vcontrol * (R23 + R24) / R24 Gain = 10V / 2.000V = 5"
- note removed: "0-12V in, 0-2.000V out"
- note removed: "ICSP"
- note removed: "Vo = Vcontrol * (R23 + R24) / R24 Gain = 12V / 2.048V = 5.86"
- moved on the sheet: C1
