File: v1/eagle/mainboard_v1.brd (EAGLE design)
At the start: 100 x 80 mm, 30 parts, among them J1 ATX24RH

Commit message: outstanding work
Parts:
- removed CAP_BUTTONS: (no value), con-amp-quick:04P
- removed FIXED_BREAKOUT: (no value), con-amp-quick:05P
- removed MAINSLED, POWERSWITCH: M02PTH, SparkFun-Connectors:1X02
- removed R4, R5, R6, R7: (no value), rcl:R0805
- removed RV1: (no value), SparkFun-Electromechanical:TRIM_POT
- removed T1, T2, T3: (no value), transistor:SOT23-BEC
- added -12V_OUT, 12V_OUT, 3V3_OUT, 5V_OUT, GND_FIX: TPPAD1-20, testpad:P1-20
- added CH1, CH2: (no value), led:LED5MM
- added I2C_EXTRA, JP1: M05X2NO_SILK, SparkFun-Connectors:2X5_NOSILK
- added LD1, LD2, LD3, LD4: (no value), led:DUOLED-A-5MM
- added PWRGOOD, PWRSW, STANDBY: M02PTH, SparkFun-Connectors:1X02
- added Q1, Q2, QA1, QA2, QA3, QB1, QB2, QB3, QC1, QC2, QC3, QD1, QD2, QD3: 2N7002L, parts:SOT23
- added QD4, QD5: BSS84, transistor-small-signal:SOT23
- added R12, RB1, RB2, RB3, RB4, RC1, RC2, RC3, RC4, RD1, RD2, RD3, RD4, RD5: (no value), rcl:R0805
- added R13: 1R1 10W, resistor-power:MNS-5
- added RA1: 10k, rcl:R0805
- added RA2: 470, rcl:R0805
- added RA3, RA4: 1M, rcl:R0805
- added U$1, U$3, U$4, U$5: MF-R300, parts:MR-300
- added U$10, U$6, U$8, U$9: SPST, parts:2P_REMOTE
- LCD: device con-amp-quick:12P -> con-amp-quick:04P
- U$2: value ARDUINO_UNO_R3 -> ARDUINO_UNO_R3MINIMUM; device parts:ARDUINO_UNO_R3 -> parts:ARDUINO_UNO_R3_MIN
- moved R2 34.8 mm to (21.0, 11.2), turned to 0 degrees
- moved R3 33.9 mm to (18.2, 13.8), turned to 180 degrees
- moved R10 21.0 mm to (65.5, 7.50), turned to 0 degrees
- moved FAN1 17.8 mm to (52.2, 62.0)
- moved FAN2 13.0 mm to (47.0, 62.0)
- moved R11 11.3 mm to (59.0, 7.50), turned to 0 degrees
- moved R9 11.3 mm to (45.0, 43.0)
- moved R8 11.0 mm to (47.5, 43.0)
- moved R1 7.60 mm to (81.5, 4.25), turned to 0 degrees
- moved SPKR 7.50 mm to (42.5, 62.0), turned to 180 degrees
- moved J1 4.00 mm to (94.5, 40.0)
- moved LCD 1.95 mm to (21.5, 76.2), turned to 0 degrees
- moved ROTARY 1.75 mm to (7.75, 67.8)
- moved C1 1.35 mm to (32.5, 58.0)
- moved U$2 0.25 mm to (0.00, 53.5)
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Connections:
- removed net A2: R6.2, U$2.A2
- removed net A3: R7.2, U$2.A3
- removed net N$11: CAP_BUTTONS.4, R4.1
- removed net N$12: CAP_BUTTONS.3, R5.1
- removed net N$6: LCD.3, RV1.1
- new net 5V_OUT: 5V_OUT.TP, QB2.1, QB3.1, RB4.1, U$3.P$2
- new net 5V_OUT1: 3V3_OUT.TP, QC2.1, QC3.1, RC4.1, U$4.P$2
- new net 5V_STANDBY: J1.9, R1.2
- new net CH1_SW: CH1.K, U$2.A3
- new net CH2_SW: CH2.K, U$2.A2
- new net D13: JP1.1, U$2.D13
- new net N$18: PWRGOOD.2, R12.1
- new net N$20: RA1.1, U$1.P$2, U$6.2
- new net N$21: LD3.CR, QC1.3
- new net N$22: LD3.A, RC2.1
- new net N$23: LD3.CX, QC2.3
- new net N$24: QD1.1, QD3.3, RD1.2, RD3.1
- new net N$25: QD5.3, RD1.1
- new net N$26: LD4.CR, QD1.3
- new net N$27: 12V_OUT.TP, QA2.1, QA3.1, RA4.1, U$1.P$1
- new net N$28: QB1.1, QB3.3, RB1.2, RB3.1
- new net N$29: RB1.1, U$3.P$1, U$8.2
- new net N$30: LD4.A, RD2.1
- new net N$31: QA1.1, QA3.3, RA1.2, RA3.1
- new net N$32: LD4.CX, QD2.3
- new net N$33: QC1.1, QC3.3, RC1.2, RC3.1
- new net N$34: RC1.1, U$4.P$1, U$9.2
- new net N$36: -12V_OUT.TP, QD4.1, U$5.P$2
- new net N$39: QD5.1, RD5.1, U$10.2, U$5.P$1
- new net N$40: QD2.1, QD3.1, QD4.3, RD4.1
- new net N$9: LD2.A, RB2.1
- net +12V: now also U$6.1; no longer FIXED_BREAKOUT.5
- net +3V3: now also U$9.1; no longer FIXED_BREAKOUT.3
- net +5V: now also LCD.4, QD4.2, QD5.2, R10.1, R11.1, R13.1, RA2.2, RB2.2, RC2.2, RD2.2, RD5.2, U$8.1; no longer FIXED_BREAKOUT.4, LCD.11, LCD.2, RV1.3
- net -12V: now also U$10.1; no longer FIXED_BREAKOUT.1
- net A0: no longer R4.2
- net A1: no longer R5.2
- net FAN_CTRL: now also Q2.1, R2.2; no longer R2.1, R3.1
- net GNDA: now also GND_FIX.TP, JP1.10, JP1.2, JP1.4, JP1.6, JP1.8, LCD.3, PWRGOOD.1, PWRSW.1, Q1.2, Q2.2, QA1.2, QA2.2, QA3.2, QB1.2, QB2.2, QB3.2, QC1.2, QC2.2, QC3.2, QD1.2, QD2.2, QD3.2, R13.2, R2.1, R3.1, RA3.2, RA4.2, RB3.2, RB4.2, RC3.2, RC4.2, RD3.2, RD4.2, STANDBY.1; no longer FIXED_BREAKOUT.2, LCD.1, LCD.12, LCD.5, MAINSLED.1, POWERSWITCH.1, R11.1, RV1.2, T1.E, T2.E
- net LCD_DB4: no longer LCD.7
- net LCD_DB5: no longer LCD.8
- net LCD_DB6: no longer LCD.9
- net LCD_DB7: no longer LCD.10
- net LCD_E: no longer LCD.6
- net LCD_RS: no longer LCD.4
- net N$1: now also FAN1.1, FAN2.1, Q2.3; no longer R2.2, T1.B
- net N$13: now also LD1.A, RA2.1; no longer CAP_BUTTONS.2, R6.1
- net N$14: now also LD1.CX, QA2.3; no longer CAP_BUTTONS.1, R7.1
- net N$15: now also LD1.CR, QA1.3; no longer SPKR.1, T3.C
- net N$16: now also LD2.CX, QB2.3; no longer R10.2, T3.B
- net N$17: now also LD2.CR, QB1.3; no longer R11.2, T3.E
- net N$2: now also STANDBY.2; no longer MAINSLED.2
- net N$3: now also Q1.3, SPKR.1; no longer R3.2, T2.B
- net N$4: now also CH1.A, R10.2; no longer FAN1.1, T1.C
- net N$5: now also CH2.A, R11.2; no longer FAN2.1, T2.C
- net POWER_GOOD: now also R12.2; no longer R1.2
- net POWER_ON: now also PWRSW.2; no longer POWERSWITCH.2
- net SCL: now also I2C_EXTRA.1, I2C_EXTRA.3, I2C_EXTRA.5, I2C_EXTRA.7, I2C_EXTRA.9, LCD.1
- net SDA: now also I2C_EXTRA.10, I2C_EXTRA.2, I2C_EXTRA.4, I2C_EXTRA.6, I2C_EXTRA.8, LCD.2
- net SPKR: now also Q1.1, R3.2; no longer R10.1
Routing:
- net CH2_SW: track 0.00 -> 132.1 mm, vias 0 -> 1
- net +5V: track 328.7 -> 432.3 mm, vias 3 -> 4
- net LCD_E: track 86.2 -> 0.00 mm
- net LCD_DB4: track 86.0 -> 0.00 mm
- net LCD_RS: track 85.6 -> 0.00 mm
- net LCD_DB5: track 83.5 -> 0.00 mm
- net LCD_DB7: track 82.9 -> 0.00 mm
- net LCD_DB6: track 82.9 -> 0.00 mm
- net FAN_CTRL: track 11.4 -> 91.9 mm, vias 0 -> 2
- net N$4: track 79.5 -> 2.63 mm, vias 4 -> 0
- net 5V_OUT: track 0.00 -> 75.3 mm
- net N$5: track 71.2 -> 2.53 mm, vias 3 -> 0
- net D13: track 0.00 -> 62.6 mm
- net N$12: track 57.3 -> 0.00 mm
- net N$29: track 0.00 -> 57.2 mm
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- removed copper zone on layer 1, net GNDA
- removed copper zone on layer 16, net GNDA
Other:
- board text added: "A0"
- board text added: "D13"
- board text removed: "+12"
- board text removed: "+5"
- board text removed: "-12"
- board text removed: "3V3"
- board text removed: "GND"
